Commit message: add description to support Gazebo

File: robot/toio.urdf.xacro (robot description, xacro)
@@ -1,7 +1,28 @@
 <?xml version="1.0"?>
 <robot name="toio" xmlns:xacro="http://ros.org/wiki/xacro">
+  <!-- Inertial -->
+  <xacro:macro name="inertial_box" params="mass height width depth">
+    <mass value="${mass}"/>
+    <inertia ixx="${(mass*(width*width+depth*depth))/12}" ixy="0" ixz="0"
+      iyy="${(mass*(height*height+depth*depth))/12}" iyz="0"
+      izz="${(mass*(height*height+width*width))/12}" />
+  </xacro:macro>
+  <xacro:macro name="inertial_cylinder" params="mass radius length">
+    <mass value="${mass}"/>
+    <inertia ixx="${((radius*radius)/4 + (length*length)/12)*mass}" ixy="0" ixz="0"
+      iyy="${((radius*radius)/4 + (length*length)/12)*mass}" iyz="0"
+      izz="${(mass*radius*radius)/2}" />
+  </xacro:macro>
+  <xacro:macro name="inertial_sphere" params="mass radius">
+    <inertial>
+      <mass value="${mass}" />
+      <inertia ixx="${(2/5) * mass * radius * radius}" ixy="0.0" ixz="0.0"
+               iyy="${(2/5) * mass * radius * radius}" iyz="0.0"
+               izz="${(2/5) * mass * radius * radius}" />
+    </inertial>
+  </xacro:macro>
   <!-- center -->
   <link name="center">
-      <visual>
+    <visual>
       <origin xyz="0 0 0" rpy="3.14159 0 0"/>
       <geometry>
@@ -12,18 +33,163 @@
       </material>
     </visual>
+    <collision>
+      <origin xyz="0 0 0.0125" rpy="0 0 0" />
+      <geometry>
+        <box size="0.0318 0.0318 0.025"/>
+      </geometry>
+    </collision>
+    <inertial>
+      <origin xyz="0 0 0.0125"/>
+      <xacro:inertial_box mass="0.2" height="0.0256" width="0.0318" depth="0.0318"/>
+    </inertial>
   </link>
+  <joint name="base_footprint_joint" type="fixed">
+    <parent link="center" />
+    <child link="base_footprint" />
+    <origin xyz="0.0038 0 0" rpy="0 0 0"/>
+  </joint>
+  <!-- base_footprint -->
+  <link name="base_footprint" />
   <joint name="base_link_joint" type="fixed">
-    <parent link="center" />
+    <parent link="base_footprint" />
     <child link="base_link" />
-    <origin xyz="0.0038 0 0.00625" rpy="0 0 0"/>
+    <origin xyz="0 0 0.00625" rpy="0 0 0"/>
   </joint>
   <!-- base_link -->
   <link name="base_link" />
-  <joint name="base_footprint_joint" type="fixed">
+  <!-- Wheel(right) -->
+  <joint name="base_r_drive_wheel_joint"
+        type="continuous">
     <parent link="base_link" />
-    <child link="base_footprint" />
-    <origin xyz="0 0 -0.00625" rpy="0 0 0"/>
+    <child link="base_r_drive_wheel_link" />
+    <origin xyz="0.0 -0.0133 0.0" rpy="-1.57 0 0" />
+    <axis xyz="0 0 1" />
   </joint>
-  <!-- base_footprint -->
-  <link name="base_footprint" />
+  <link name="base_r_drive_wheel_link">
+    <inertial>
+      <mass value="0.2" />
+      <origin xyz="0 0 0" rpy="0 0 0" />
+      <xacro:inertial_cylinder mass="0.2"
+          radius="0.00625" length="0.002"/>
+    </inertial>
+    <visual>
+      <origin xyz="0 0 0" rpy="0 0 0" />
+      <geometry>
+        <cylinder radius="0.00625" length="0.002" />
+      </geometry>
+      <material name="wheel">
+        <color rgba="0.5 0.5 0.5 1.0" />
+      </material>
+    </visual>
+    <collision>
+      <origin xyz="0 0 0" rpy="0 0 0" />
+      <geometry>
+        <cylinder radius="0.00625" length="0.002" />
+      </geometry>
+    </collision>
+  </link>
+  <gazebo reference="base_r_drive_wheel_link">
+    <mu1>1.0</mu1>
+    <mu2>1.0</mu2>
+    <kp>1e+5</kp>
+    <kd>1.0</kd>
+  </gazebo>
+  <!-- Wheel(left) -->
+  <joint name="base_l_drive_wheel_joint"
+        type="continuous">
+    <parent link="base_link" />
+    <child link="base_l_drive_wheel_link" />
+    <origin rpy="-1.57 0 0"
+            xyz="0.0 0.0133 0.0" />
+    <axis xyz="0 0 1" />
+  </joint>
+  <link name="base_l_drive_wheel_link">
+    <inertial>
+      <mass value="0.2" />
+      <origin xyz="0 0 0" rpy="0 0 0" />
+      <xacro:inertial_cylinder mass="0.2"
+          radius="0.00625" length="0.002"/>
+    </inertial>
+    <visual>
+      <origin xyz="0 0 0" rpy="0 0 0" />
+      <geometry>
+        <cylinder radius="0.00625" length="0.002" />
+      </geometry>
+      <material name="wheel">
+        <color rgba="0.5 0.5 0.5 1.0" />
+      </material>
+    </visual>
+    <collision>
+      <origin xyz="0 0 0" rpy="0 0 0" />
+      <geometry>
+        <cylinder radius="0.00625" length="0.002" />
+      </geometry>
+    </collision>
+  </link>
+  <gazebo reference="base_l_drive_wheel_link">
+    <mu1>1.0</mu1>
+    <mu2>1.0</mu2>
+    <kp>1e+5</kp>
+    <kd>1.0</kd>
+  </gazebo>
+  <gazebo>
+      <plugin
+        filename="gz-sim-diff-drive-system"
+        name="gz::sim::systems::DiffDrive">
+        <left_joint>base_l_drive_wheel_joint</left_joint>
+        <right_joint>base_r_drive_wheel_joint</right_joint>
+        <wheel_separation>0.0266</wheel_separation>
+        <wheel_radius>0.00625</wheel_radius>
+        <max_linear_acceleration>0.35</max_linear_acceleration>
+        <min_linear_acceleration>-0.35</min_linear_acceleration>
+        <max_angular_acceleration>26.17994</max_angular_acceleration>
+        <min_angular_acceleration>-26.17994</min_angular_acceleration>
+        <max_linear_velocity>1.6</max_linear_velocity>
+        <min_linear_velocity>-1.6</min_linear_velocity>
+        <max_angular_velocity>3.0</max_angular_velocity>
+        <min_angular_velocity>-3.0</min_angular_velocity>
+        <topic>/cmd_vel</topic>
+        <odom_topic>/odom</odom_topic>
+        <tf_topic>tf</tf_topic>
+        <frame_id>odom</frame_id>
+        <child_frame_id>base_footprint</child_frame_id>
+        <odom_publish_frequency>10</odom_publish_frequency>
+      </plugin>
+      <plugin
+        filename="gz-sim-joint-state-publisher-system"
+        name="gz::sim::systems::JointStatePublisher">
+        <topic>/joint_states</topic>
+        <update_rate>30</update_rate>
+      </plugin>
+  </gazebo>
+  <joint name="rear_caster_joint" type="fixed">
+    <parent link="base_footprint"/>
+    <child link="rear_caster_link"/>
+    <origin xyz="-0.0149 0 0.001" rpy="0 0 0" />
+  </joint>
+  <link name="rear_caster_link">
+    <visual>
+      <geometry>
+        <sphere radius="0.001"/>
+      </geometry>
+      <material name="caster">
+        <color rgba="1.0 1.0 1.0 1.0" />
+      </material>
+    </visual>
+    <collision>
+      <geometry>
+        <sphere radius="0.001"/>
+      </geometry>
+    </collision>
+    <xacro:inertial_sphere mass="0.01" radius="0.001"/>
+  </link>
+  <gazebo reference="rear_caster_joint">
+    <preserveFixedJoint>true</preserveFixedJoint>
+  </gazebo>
+  <gazebo reference="rear_caster_link">
+    <mu1>0.0</mu1>
+    <mu2>0.0</mu2>
+    <kp>1000000.0</kp>
+    <kd>1.0</kd>
+  </gazebo>
 </robot>
