Commit message: add an indicator LED to the toio model
The LED is a visual on the lower front of the cube, where the indicator of
the real cube sits. It is driven in Gazebo by the ToioLedSystem plugin of
toio_gazebo, which subscribes to /model/<robot_name>/led, so that the cube
can be lit through the same interface as the real one.

The fixed joint of the LED is lumped into "center" when the URDF is
converted to SDF, which rewrites the visual name into a generated one. The
plugin therefore matches the visual by the substring "led", and test_urdf.py
guards that nothing else in the model matches that substring.

Co-Authored-By: Claude Opus 5 (1M context) <noreply@anthropic.com>

File: robot/toio.urdf.xacro (robot description, xacro)
@@ -4,4 +4,8 @@
        so that multiple instances can be spawned without sharing topics -->
   <xacro:arg name="robot_name" default="toio"/>
+  <!-- Lighting time of the indicator LED in milliseconds. 0 keeps the LED lit
+       until the next command, 10-2550 lets the cube turn it off on its own.
+       This mirrors the led_duration_ms parameter of the toio_ros2 node. -->
+  <xacro:arg name="led_duration_ms" default="0"/>
   <!-- Inertial -->
   <xacro:macro name="inertial_box" params="mass height width depth">
@@ -45,4 +49,30 @@
       <origin xyz="0 0 0.0125"/>
       <xacro:inertial_box mass="0.2" height="0.0256" width="0.0318" depth="0.0318"/>
+    </inertial>
+  </link>
+  <!-- Indicator LED.
+       The cube body spans x/y of +-0.0159 and z of 0 to 0.02425 in the frame
+       of "center", so this sits on the lower part of the front face, where the
+       indicator of the real cube is. The visual is named "led" because the
+       ToioLedSystem plugin looks the entity up by that substring. The fixed
+       joint below is lumped into "center" when the URDF is converted to SDF,
+       which rewrites the visual name into a longer generated one. -->
+  <joint name="led_joint" type="fixed">
+    <parent link="center"/>
+    <child link="led_link"/>
+    <origin xyz="0.0160 0 0.005" rpy="0 0 0"/>
+  </joint>
+  <link name="led_link">
+    <visual name="led">
+      <geometry>
+        <box size="0.0018 0.010 0.004"/>
+      </geometry>
+      <material name="led_off">
+        <color rgba="0.15 0.15 0.15 1.0"/>
+      </material>
+    </visual>
+    <inertial>
+      <mass value="1e-6"/>
+      <inertia ixx="1e-9" ixy="0" ixz="0" iyy="1e-9" iyz="0" izz="1e-9"/>
     </inertial>
   </link>
@@ -175,4 +205,11 @@
         <update_frequency>50</update_frequency>
       </plugin>
+      <plugin
+        filename="ToioLedSystem"
+        name="toio_gazebo::ToioLedSystem">
+        <topic>/model/$(arg robot_name)/led</topic>
+        <led_visual>led</led_visual>
+        <led_duration_ms>$(arg led_duration_ms)</led_duration_ms>
+      </plugin>
   </gazebo>
   <joint name="rear_caster_joint" type="fixed">

Commit message: put the lamp where the specification puts it
https://toio.github.io/toio-spec/docs/ble_light/ gives the cube one lamp on
its bottom, and the parts diagram of
https://toio.github.io/toio-spec/docs/hardware_components/ shows it as the
ball at the rear of the underside that doubles as the function button. The
lamp was on the front face before, which is not where it is on the cube.

Fitting a sphere to that ball in the mesh puts it 11.108 mm behind "center"
with a radius of 3.49 mm, which agrees with the 11.1 mm of the bottom view
drawing, so the visual is now a sphere there instead of a box on the front.
It is 3.7 mm rather than 3.49 mm because the ball in the mesh is not
perfectly round and reaches 3.62 mm from that centre, which would otherwise
poke through the lamp where it shows.

Only the cap below the flat underside of the body shows, so the lamp is best
seen from a low angle, as on the real cube.

Co-Authored-By: Claude Opus 5 (1M context) <noreply@anthropic.com>

File: robot/toio.urdf.xacro (robot description, xacro)
@@ -51,23 +51,32 @@
     </inertial>
   </link>
-  <!-- Indicator LED.
-       The cube body spans x/y of +-0.0159 and z of 0 to 0.02425 in the frame
-       of "center", so this sits on the lower part of the front face, where the
-       indicator of the real cube is. The visual is named "led" because the
-       ToioLedSystem plugin looks the entity up by that substring. The fixed
-       joint below is lumped into "center" when the URDF is converted to SDF,
-       which rewrites the visual name into a longer generated one. -->
+  <!-- Indicator lamp.
+       https://toio.github.io/toio-spec/docs/ble_light/ gives the cube one lamp
+       on its bottom, and the parts diagram of
+       https://toio.github.io/toio-spec/docs/hardware_components/ shows it as
+       the ball at the rear that doubles as the function button. Fitting a
+       sphere to that ball in the mesh gives a radius of 3.49 mm around
+       (-11.1, 0, 3.28) mm in the frame of "center", which agrees with the
+       11.1 mm of the bottom view drawing. The flat part of the underside is at
+       z = 1.66 mm, so only the cap below that shows, as on the real cube.
+       The ball in the mesh is not perfectly round, reaching 3.62 mm from that
+       centre, so the sphere here is 3.7 mm to cover it everywhere it shows
+       instead of letting the mesh poke through it.
+       The visual is named "led" because the ToioLedSystem plugin looks the
+       entity up by that substring. The fixed joint below is lumped into
+       "center" when the URDF is converted to SDF, which rewrites the visual
+       name into a longer generated one. -->
   <joint name="led_joint" type="fixed">
     <parent link="center"/>
     <child link="led_link"/>
-    <origin xyz="0.0160 0 0.005" rpy="0 0 0"/>
+    <origin xyz="-0.0111 0 0.0033" rpy="0 0 0"/>
   </joint>
   <link name="led_link">
     <visual name="led">
       <geometry>
-        <box size="0.0018 0.010 0.004"/>
+        <sphere radius="0.0037"/>
       </geometry>
       <material name="led_off">
-        <color rgba="0.15 0.15 0.15 1.0"/>
+        <color rgba="0.8 0.8 0.8 1.0"/>
       </material>
     </visual>

Commit message: Add IMU sensor and wheel odometry to the sim cube
Mirror the topics toio_ros2 added (#48/#49/#51) on the simulation side:

- Add an IMU sensor on the "center" link (behind /toio/imu), rate driven by
  the new imu_interval_ms arg. Needs the gz-sim-imu-system in the world.
- Wire the DiffDrive wheel odometry to /model/<robot_name>/odom as odom ->
  center at 20Hz (was a dummy topic), for the new /odom.
- Add a frame_prefix arg so the odometry/IMU frame ids carry the multi-cube
  prefix (robot_state_publisher cannot rewrite these plugin-emitted frames).

Consumed by toio_gazebo (bridge + launch).

Co-Authored-By: Claude Opus 4.8 (1M context) <noreply@anthropic.com>
Claude-Session: https://claude.ai/code/session_01RoihHEqf5aYbFVLhrHD2FH

File: robot/toio.urdf.xacro (robot description, xacro)
@@ -11,4 +11,14 @@
        lighting up only itself, without casting color on the mat. -->
   <xacro:arg name="led_light_intensity" default="1.0"/>
+  <!-- Prefix of the TF frames (e.g. "toio1/") for multi-cube setups. The
+       DiffDrive odometry and the IMU sensor emit frame ids as plain strings,
+       so the prefix has to be baked into the model here (robot_state_publisher
+       cannot rewrite them the way it does the URDF link frames). -->
+  <xacro:arg name="frame_prefix" default=""/>
+  <!-- Notification interval of the posture angle behind /toio/imu, in
+       milliseconds. Mirrors the imu_interval_ms parameter of toio_ros2; the
+       IMU sensor update rate below is 1000/imu_interval_ms Hz. -->
+  <xacro:arg name="imu_interval_ms" default="100"/>
+  <xacro:property name="imu_interval_ms" value="$(arg imu_interval_ms)"/>
   <!-- Inertial -->
   <xacro:macro name="inertial_box" params="mass height width depth">
@@ -223,9 +233,14 @@
         <min_angular_velocity>-26.17994</min_angular_velocity>
         <topic>/model/$(arg robot_name)/cmd_vel</topic>
-        <odom_topic>/odom_dummy</odom_topic>
+        <!-- Wheel odometry, mirroring toio_ros2's /odom (odom -> center) at
+             20Hz. Only the odometry message is published here; the tf tree is
+             provided by the launch (map -> odom -> center, with map -> center
+             kept at the mat-perfect ground-truth pose), so tf_topic stays a
+             dummy that nothing subscribes to. -->
+        <odom_topic>/model/$(arg robot_name)/odom</odom_topic>
         <tf_topic>tf_dummy</tf_topic>
-        <frame_id>odom_dummy</frame_id>
-        <child_frame_id>base_footprint</child_frame_id>
-        <odom_publish_frequency>10</odom_publish_frequency>
+        <frame_id>$(arg frame_prefix)odom</frame_id>
+        <child_frame_id>$(arg frame_prefix)center</child_frame_id>
+        <odom_publish_frequency>20</odom_publish_frequency>
       </plugin>
       <plugin
@@ -255,4 +270,18 @@
       </plugin>
   </gazebo>
+  <!-- IMU behind /toio/imu (mirrors toio_ros2 #51). Attached to the cube body
+       frame "center". Gazebo fills orientation, angular velocity and linear
+       acceleration; the real cube only reports orientation, but the sim value
+       is bridged as-is (see toio_gazebo README). The update rate follows
+       imu_interval_ms (1000/imu_interval_ms Hz, default 10Hz). Needs the
+       gz-sim-imu-system in the world. -->
+  <gazebo reference="center">
+    <sensor name="imu" type="imu">
+      <topic>/model/$(arg robot_name)/imu</topic>
+      <gz_frame_id>$(arg frame_prefix)center</gz_frame_id>
+      <update_rate>${1000.0 / imu_interval_ms}</update_rate>
+      <always_on>1</always_on>
+    </sensor>
+  </gazebo>
   <joint name="rear_caster_joint" type="fixed">
     <parent link="base_footprint"/>
